File: voice_card.sch (KiCad schematic (older format))
At the start: 207 parts, among them J1 PCI_11_49, Q1 MMBF4391LT1G, Q10 DMMT3906, Q11 BC857BS, Q2 2N3904, Q3 BCM847, Q4 DMMT3904, Q5 DMMT3906, Q6 MMBF4391LT1G, Q7 BCM847, Q8 2N3904, Q9 DMMT3904, U1 TL074-, U10 TL072-, U11 TL074-, U12 NE555, U13 LM311M, U14 CD4052, U15 TL072-, U16 TL072-, U17 LM13700, U18 LM13700, U19 LM13700, U2 TL074-, U20 TL072-, U3 NE555, U4 LF351, U5 TL072-, U6 LM311M, U7 CD4052, U8 TL074-, U9 LF351

Commit message: EG2 placed and routed
Connections:
- net GND: now also Q10.1; no longer Q10.2
- net at C28.2, Q9.6, R93.1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: now also Q10.6; no longer Q10.3
- net at Q9.4, Q9.5, R86.2: now also Q10.4, Q10.5; no longer Q10.4, Q10.5
- net at C27.2, Q9.3, U11.6 (-): now also Q10.3; no longer Q10.6
- net at R88.2, R90.2, R91.2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: now also Q10.2; no longer Q10.1
